File: RC1802 SBC/RC1802 SBC.sch (KiCad schematic (older format))
At the start: 66 parts, among them J1 CONN_01X39, J2 BARREL_JACK, SW1 RUN, SW10 IN5, SW11 IN6, SW12 IN7, SW2 IN, SW3 MP, SW4 RUN, SW5 IN0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

Commit message: Added switches.
Parts:
- AFF1, AFF2: footprint (none) -> Displays_7-Segment:7SegmentLED_LTS6760_LTS6780
- C1, C10, C2, C3, C4, C5, C6, C7, C8, C9: footprint (none) -> Capacitors_THT:C_Disc_D4.7mm_W2.5mm_P5.00mm
- D1: value LED -> Q LED; footprint (none) -> LEDs:LED_D5.0mm
- D2, D3, D4, D5, D6, D7: footprint (none) -> Diodes_THT:D_DO-35_SOD27_P7.62mm_Horizontal
- J2: footprint (none) -> Connectors:BARREL_JACK
- JP1, JP3, JP4: footprint (none) -> Pin_Headers:Pin_Header_Straight_1x03_Pitch2.54mm
- JP2: footprint (none) -> Pin_Headers:Pin_Header_Straight_1x02_Pitch2.54mm
- R1, R10, R11, R12, R13, R14, R15, R16, R17, R2, R3, R4, R5, R6, R7, R8, R9: footprint (none) -> Resistors_THT:R_Axial_DIN0207_L6.3mm_D2.5mm_P10.16mm_Horizontal
- SW1, SW10, SW11, SW12, SW3, SW4, SW5, SW6, SW7, SW8, SW9: footprint (none) -> switches:SPDT_SWITCH
- SW2: footprint (none) -> switches:SPDT_PUSH
- U1, U12: footprint (none) -> Housings_DIP:DIP-32_W15.24mm_Socket
- U10, U5, U8: footprint (none) -> Housings_DIP:DIP-16_W7.62mm_Socket
- U2, U9: footprint (none) -> Housings_DIP:DIP-20_W7.62mm_Socket
- U3: footprint DIP28 -> Housings_DIP:DIP-32_W15.24mm_Socket
- U4, U6, U7: footprint (none) -> Housings_DIP:DIP-14_W7.62mm_Socket
Connections:
- no-connect marks 9 -> 10

Commit message: Ran out of space :(
Parts:
- removed R11, R12, R13, R14, R15, R16, R17: 100k, Resistors_THT:R_Axial_DIN0207_L6.3mm_D2.5mm_P10.16mm_Horizontal, symbol R
- added C11: 100nF, Capacitors_THT:C_Disc_D4.7mm_W2.5mm_P5.00mm, symbol C_Small
- added J3, J4, J5, J6: Mount, mounting:1pin, symbol CONN_01X01
- added RN1: 100k, Resistors_THT:R_Array_SIP9, symbol R_Network08
- AFF1: value LTS-6980HR -> MSB
- AFF2: value LTS-6980HR -> LSB
- R10: value 100k -> 470
- SW1: value RUN -> CLEAR
- SW4: value RUN -> WAIT
- U1: footprint Housings_DIP:DIP-32_W15.24mm_Socket -> Housings_DIP:DIP-40_W15.24mm_Socket
- renumbered U12 to U11
Connections:
- net DMA_IN: now also J1.36 (P36); no longer J1.38 (P38)
- net DMA_OUT: now also J1.35 (P35); no longer J1.39 (P39)
- net GND: now also C11.2
- net LOAD: no longer D3.2 (A), U1.2 (~WAIT~), U4.11, U4.6
- net N0: now also J1.39 (P39); no longer J1.35 (P35)
- net N1: now also J1.38 (P38); no longer J1.36 (P36)
- net RUN: no longer SW1.2 (B), U1.3 (~CLEAR), U5.2, U5.3
- net VCC: now also C11.1, RN1.1 (common); no longer D1.2 (A)
- net at R10.1: now also D1.2 (A); no longer SW5.3 (C)
- net at SW6.3 (C): now also RN1.8 (R7)
- net at SW7.3 (C): now also RN1.7 (R6)
- net at SW8.3 (C): now also RN1.6 (R5)
- net at SW9.3 (C): now also RN1.5 (R4)
- net at SW10.3 (C): now also RN1.4 (R3)
- net at SW11.3 (C): now also RN1.3 (R2)
- net at SW12.3 (C): now also RN1.2 (R1)
- new net: RN1.9 (R8), SW5.3 (C)
- new net CLEAR: SW1.2 (B), U1.3 (~CLEAR), U5.2, U5.3
- new net WAIT: D3.2 (A), U1.2 (~WAIT~), U4.11, U4.6
- no-connect marks 10 -> 15
