File: RC1802 CPU/RC1802 CPU.kicad_pcb (KiCad board)
At the start: 2 copper layers, 99.1 x 99.1 mm, 65 parts, among them J1 CONN_01X39, J2 BARREL_JACK, J3 Mount, J4 Mount, J5 Mount, J6 Mount, SW1 CLEAR, SW10 IN5, SW11 IN6, SW12 IN7, SW2 IN, SW3 MP, SW4 WAIT, SW5 IN0, SW6 IN1, SW7 IN2, SW8 IN3, SW9 IN4, U1 CDP1802, U10 MC14495P1, U11 28C256, U2 74LS373, U3 HM62256BLP-7, U4 74LS04, U5 4050, U6 4013, U7 74LS10, U8 MC14495P1, U9 74LS245, X1 CXO_DIP14

Commit message: Placed PCB components (no tracks)
Parts:
- removed AFF1: MSB, Displays_7-Segment:7SegmentLED_LTS6760_LTS6780
- removed AFF2: LSB, Displays_7-Segment:7SegmentLED_LTS6760_LTS6780
- removed C10, C11, C7, C8, C9: 100nF, Capacitors_THT:C_Disc_D4.7mm_W2.5mm_P5.00mm
- removed RN1: 100k, Resistors_THT:R_Array_SIP9
- removed SW1: CLEAR, switches:SPDT_SWITCH
- removed SW10: IN5, switches:SPDT_SWITCH
- removed SW11: IN6, switches:SPDT_SWITCH
- removed SW12: IN7, switches:SPDT_SWITCH
- removed SW2: IN, switches:SPDT_PUSH
- removed SW3: MP, switches:SPDT_SWITCH
- removed SW4: WAIT, switches:SPDT_SWITCH
- removed SW5: IN0, switches:SPDT_SWITCH
- removed SW6: IN1, switches:SPDT_SWITCH
- removed SW7: IN2, switches:SPDT_SWITCH
- removed SW8: IN3, switches:SPDT_SWITCH
- removed SW9: IN4, switches:SPDT_SWITCH
- removed U10, U8: MC14495P1, Housings_DIP:DIP-16_W7.62mm_Socket
- removed U11: 28C256, Housings_DIP:DIP-32_W15.24mm_Socket
- removed U7: 74LS10, Housings_DIP:DIP-14_W7.62mm_Socket
- removed U9: 74LS245, Housings_DIP:DIP-20_W7.62mm_Socket
- added D8: LED_Small, LEDs:LED_D5.0mm, F.Cu at (177.8, 50.8)
- added J7: BARREL_JACK, Connectors:BARREL_JACK, F.Cu at (110.5, 57.1)
- added JP5: SLOT1_WE, Pin_Headers:Pin_Header_Straight_1x03_Pitch2.54mm, F.Cu at (160.0, 83.8)
- added JP6: BM_OE, Pin_Headers:Pin_Header_Straight_1x03_Pitch2.54mm, F.Cu at (141.0, 77.5)
- added R11: 220, Resistors_THT:R_Axial_DIN0207_L6.3mm_D2.5mm_P10.16mm_Horizontal, F.Cu at (177.8, 74.9)
- added R12: 220, Resistors_THT:R_Axial_DIN0207_L6.3mm_D2.5mm_P10.16mm_Horizontal, F.Cu at (181.0, 74.9)
- added R13: 220, Resistors_THT:R_Axial_DIN0207_L6.3mm_D2.5mm_P10.16mm_Horizontal, F.Cu at (184.2, 74.9)
- added R14: 220, Resistors_THT:R_Axial_DIN0207_L6.3mm_D2.5mm_P10.16mm_Horizontal, F.Cu at (187.3, 74.9)
- added R15: 220, Resistors_THT:R_Axial_DIN0207_L6.3mm_D2.5mm_P10.16mm_Horizontal, F.Cu at (190.5, 74.9)
- D1: value Q LED -> LED_Small
- D2, D3, D4, D5, D6, D7: value 1N4848 -> LED_Small; footprint Diodes_THT:D_DO-35_SOD27_P7.62mm_Horizontal -> LEDs:LED_D5.0mm
- J1: value CONN_01X39 -> Mount; footprint Pin_Headers:Pin_Header_Angled_1x39_Pitch2.54mm -> mounting:1pin
- J2: value BARREL_JACK -> Mount; footprint Connectors:BARREL_JACK -> mounting:1pin
- J5: value Mount -> CONN_01X39; footprint mounting:1pin -> Pin_Headers:Pin_Header_Angled_1x39_Pitch2.54mm
- J6: value Mount -> CONN_02X20; footprint mounting:1pin -> Pin_Headers:Pin_Header_Straight_2x20_Pitch2.54mm
- JP1: value U12 WE -> Enable; footprint Pin_Headers:Pin_Header_Straight_1x03_Pitch2.54mm -> Pin_Headers:Pin_Header_Straight_1x02_Pitch2.54mm
- JP2: value Enable -> HI; footprint Pin_Headers:Pin_Header_Straight_1x02_Pitch2.54mm -> Pin_Headers:Pin_Header_Straight_1x03_Pitch2.54mm
- JP3: value HI -> LO
- JP4: value LO -> SLOT2_WE
- R10: value 470 -> 220
- R8, R9: value 47k -> 220
- U1: value CDP1802 -> 74LS04; footprint Housings_DIP:DIP-40_W15.24mm_Socket -> Housings_DIP:DIP-14_W7.62mm_Socket
- U2: value 74LS373 -> CDP1802; footprint Housings_DIP:DIP-20_W7.62mm_Socket -> Housings_DIP:DIP-40_W15.24mm_Socket
- U3: value HM62256BLP-7 -> 74LS240; footprint Housings_DIP:DIP-32_W15.24mm_Socket -> Housings_DIP:DIP-20_W7.62mm_Socket
- U4: value 74LS04 -> 74LS373; footprint Housings_DIP:DIP-14_W7.62mm_Socket -> Housings_DIP:DIP-20_W7.62mm_Socket
- U5: value 4050 -> SLOT-1; footprint Housings_DIP:DIP-16_W7.62mm_Socket -> Housings_DIP:DIP-32_W15.24mm_Socket
- U6: value 4013 -> SLOT-2; footprint Housings_DIP:DIP-14_W7.62mm_Socket -> Housings_DIP:DIP-32_W15.24mm_Socket
- moved JP1 285.9 mm to (109.9, 69.8)
- moved D2 262.1 mm to (129.5, 50.8), turned to 270 degrees
- moved D3 253.1 mm to (137.2, 50.8), turned to 270 degrees
- moved D4 237.3 mm to (144.8, 50.8), turned to 270 degrees
- moved R3 232.5 mm to (149.9, 139.7), turned to 90 degrees
- moved R1 226.9 mm to (141.0, 139.7), turned to 90 degrees
- moved D7 209.9 mm to (170.2, 50.8), turned to 270 degrees
- moved D6 191.6 mm to (162.6, 50.8), turned to 270 degrees
- moved R4 187.3 mm to (154.3, 139.7), turned to 90 degrees
- moved R8 180.2 mm to (168.3, 74.9), turned to 90 degrees
- moved R9 171.6 mm to (171.4, 74.9), turned to 90 degrees
- moved R5 170.4 mm to (158.8, 139.7), turned to 90 degrees
- moved D5 161.9 mm to (154.9, 50.8), turned to 270 degrees
- moved R7 161.2 mm to (167.6, 139.7), turned to 90 degrees
- moved JP3 159.5 mm to (172.1, 132.1)
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Connections:
- D1 pad 1: Net-(D1-Pad1) -> GND
- D2 pad 1: /~IN -> GND
- D2 pad 2: EF4 -> Net-(D2-Pad2)
- D3 pad 1: Net-(D3-Pad1) -> GND
- D3 pad 2: WAIT -> Net-(D3-Pad2)
- D4 pad 1: Net-(D3-Pad1) -> GND
- D4 pad 2: SC1 -> Net-(D4-Pad2)
- D5 pad 1: Net-(D5-Pad1) -> GND
- D5 pad 2: DMA_IN -> Net-(D5-Pad2)
- D6 pad 1: LOAD_N2 -> GND
- D7 pad 1: LOAD_N2 -> GND
- D7 pad 2: N2 -> Net-(D7-Pad2)
- J1 pad 1: EF1 -> (no net)
- J2 pad 1: VCC -> (no net)
- J5 pad 1: (no net) -> EF1
- JP1 pad 1: ~WE -> Net-(JP1-Pad1)
- JP1 pad 2: Net-(JP1-Pad2) -> CLOCK
- JP2 pad 1: Net-(JP2-Pad1) -> SLOT1_CS
- JP2 pad 2: CLOCK -> Net-(JP2-Pad2)
- JP3 pad 1: CS_ROM -> SLOT1_CS
- JP3 pad 2: Net-(JP3-Pad2) -> /MA15
- JP3 pad 3: CS_RAM -> SLOT2_CS
- JP4 pad 1: CS_RAM -> ~WE
- JP4 pad 2: /MA15 -> Net-(JP4-Pad2)
- JP4 pad 3: CS_ROM -> VCC
- R10 pad 1: Net-(D1-Pad2) -> Net-(R10-Pad1)
- R10 pad 2: VCC -> Net-(D3-Pad2)
- R8 pad 1: GND -> Net-(R8-Pad1)
- R8 pad 2: Net-(D3-Pad1) -> Net-(D1-Pad2)
- R9 pad 1: GND -> Net-(R9-Pad1)
- R9 pad 2: LOAD_N2 -> Net-(D2-Pad2)
- U1 pad 1: CLOCK -> /MA15
- U1 pad 10: /BUS5 -> (no net)
- U1 pad 11: /BUS4 -> GND
- U1 pad 12: /BUS3 -> (no net)
- U1 pad 13: /BUS2 -> GND
- U1 pad 14: /BUS1 -> VCC
- U1 pad 2: WAIT -> Net-(JP2-Pad2)
- U1 pad 3: CLEAR -> GND
- U1 pad 4: Q -> (no net)
- U1 pad 5: SC1 -> GND
- U1 pad 6: SC0 -> (no net)
- U1 pad 7: MRD -> GND
- U1 pad 8: /BUS7 -> (no net)
- U1 pad 9: /BUS6 -> GND
- U2 pad 1: GND -> CLOCK
- U2 pad 10: GND -> /BUS5
- U2 pad 11: TPA -> /BUS4
- U2 pad 12: /MA12 -> /BUS3
- U2 pad 13: /MA4 -> /BUS2
- U2 pad 14: /MA5 -> /BUS1
- U2 pad 15: /MA13 -> /BUS0
- U2 pad 16: /MA14 -> VCC
- U2 pad 17: /MA6 -> N2
- U2 pad 18: /MA7 -> N1
- U2 pad 19: /MA15 -> N0
- U2 pad 2: /MA8 -> (no net)
- U2 pad 20: VCC -> GND
- U2 pad 3: /MA0 -> (no net)
- U2 pad 4: /MA1 -> Q
- U2 pad 5: /MA9 -> SC1
- U2 pad 6: /MA10 -> SC0
- U2 pad 7: /MA2 -> MRD
- U2 pad 8: /MA3 -> /BUS7
- U2 pad 9: /MA11 -> /BUS6
- U3 pad 1: /MA14 -> Net-(JP6-Pad2)
- U3 pad 10: /MA0 -> GND
- U3 pad 11: /BUS0 -> SC1
- U3 pad 12: /BUS1 -> Net-(R11-Pad1)
- U3 pad 13: /BUS2 -> INTERRUPT
- U3 pad 14: GND -> Net-(R10-Pad1)
- U3 pad 15: /BUS3 -> DMA_IN
- U3 pad 16: /BUS4 -> Net-(R9-Pad1)
- U3 pad 17: /BUS5 -> DMA_OUT
- U3 pad 18: /BUS6 -> Net-(R8-Pad1)
- U3 pad 19: /BUS7 -> Net-(JP6-Pad2)
- U3 pad 2: /MA12 -> CLOCK
- U3 pad 20: CS_RAM -> VCC
- U3 pad 3: /MA7 -> Net-(R15-Pad1)
- U3 pad 4: /MA6 -> TPA
- U3 pad 5: /MA5 -> Net-(R14-Pad1)
- U3 pad 6: /MA4 -> TPB
- U3 pad 7: /MA3 -> Net-(R13-Pad1)
- U3 pad 8: /MA2 -> SC0
- U3 pad 9: /MA1 -> Net-(R12-Pad1)
- U4 pad 1: Net-(D1-Pad1) -> GND
- U4 pad 10: Net-(D6-Pad2) -> GND
- U4 pad 11: WAIT -> TPA
- U4 pad 12: Net-(JP3-Pad2) -> /MA12
- U4 pad 13: /MA15 -> /MA4
- U4 pad 14: VCC -> /MA5
- U4 pad 2: Q -> /MA8
- U4 pad 3: Net-(SW2-Pad2) -> /MA0
- U4 pad 4: /~IN -> /MA1
- U4 pad 5: Net-(D6-Pad2) -> /MA9
- U4 pad 6: WAIT -> /MA10
- U4 pad 7: GND -> /MA2
- U4 pad 8: Net-(SW2-Pad2) -> /MA3
- U4 pad 9: /~IN -> /MA11
- U5 pad 1: VCC -> /MA14
- U5 pad 10: (no net) -> /MA0
- U5 pad 11: (no net) -> /BUS0
- U5 pad 12: (no net) -> /BUS1
- U5 pad 13: (no net) -> /BUS2
- U5 pad 14: (no net) -> GND
- U5 pad 15: (no net) -> /BUS3
- U5 pad 16: (no net) -> /BUS4
- U5 pad 2: CLEAR -> /MA12
- U5 pad 3: CLEAR -> /MA7
- U5 pad 4: STROBE -> /MA6
- U5 pad 5: Net-(U5-Pad5) -> /MA5
- U5 pad 6: (no net) -> /MA4
- U5 pad 7: (no net) -> /MA3
- U5 pad 8: (no net) -> /MA2
- U5 pad 9: (no net) -> /MA1
- U6 pad 1: (no net) -> /MA14
- U6 pad 10: Net-(D3-Pad1) -> /MA0
- U6 pad 11: /~IN -> /BUS0
- U6 pad 12: Net-(D5-Pad1) -> /BUS1
- U6 pad 13: (no net) -> /BUS2
- U6 pad 14: VCC -> GND
- U6 pad 2: (no net) -> /MA12
- U6 pad 3: (no net) -> /MA7
- U6 pad 4: (no net) -> /MA6
- U6 pad 5: (no net) -> /MA5
- U6 pad 6: (no net) -> /MA4
- U6 pad 7: GND -> /MA3
- U6 pad 8: GND -> /MA2
- U6 pad 9: VCC -> /MA1
- X1 pad 8: Net-(JP2-Pad1) -> Net-(JP1-Pad1)
Routing:
- net VCC: track 329.4 -> 0.00 mm, vias 3 -> 0
- net Net-(SW5-Pad2): track 137.1 -> 0.00 mm
- net Net-(SW6-Pad2): track 127.4 -> 0.00 mm, vias 3 -> 0
- net Net-(SW7-Pad2): track 116.6 -> 0.00 mm, vias 3 -> 0
- net /BUS7: track 114.5 -> 0.00 mm, vias 5 -> 0
- net /BUS6: track 112.7 -> 0.00 mm, vias 3 -> 0
- net /BUS5: track 109.4 -> 0.00 mm, vias 3 -> 0
- net Net-(SW8-Pad2): track 105.8 -> 0.00 mm, vias 3 -> 0
- net Net-(SW9-Pad2): track 97.5 -> 0.00 mm, vias 3 -> 0
- net /BUS0: track 94.7 -> 0.00 mm, vias 2 -> 0
- net /BUS1: track 94.1 -> 0.00 mm, vias 6 -> 0
- net /BUS2: track 91.7 -> 0.00 mm, vias 4 -> 0
- net /BUS3: track 90.2 -> 0.00 mm, vias 4 -> 0
- net /BUS4: track 89.9 -> 0.00 mm, vias 6 -> 0
- net Net-(SW10-Pad2): track 86.6 -> 0.00 mm, vias 3 -> 0
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Other:
- board text added: "RC1802 Cosmac ELF CPU Board Revision A"

Commit message: All tracks layed out
Parts:
- moved C5 14.5 mm to (160.0, 94.0), turned to 270 degrees
- moved C6 14.5 mm to (183.5, 94.0), turned to 270 degrees
- moved C1 1.27 mm to (195.6, 113.0)
Connections:
- JP4 pad 1: ~WE -> VCC
- JP4 pad 3: VCC -> ~WE
Routing:
- net VCC: track 0.00 -> 400.2 mm, vias 0 -> 4
- net SC1: track 0.00 -> 213.0 mm, vias 0 -> 11
- net SC0: track 0.00 -> 207.6 mm, vias 0 -> 14
- net TPA: track 0.00 -> 198.5 mm, vias 0 -> 9
- net TPB: track 0.00 -> 175.0 mm, vias 0 -> 8
- net DMA_IN: track 0.00 -> 173.5 mm, vias 0 -> 16
- net /MA1: track 0.00 -> 168.2 mm, vias 0 -> 8
- net /MA0: track 0.00 -> 162.3 mm, vias 0 -> 5
- net /MA7: track 0.00 -> 159.1 mm, vias 0 -> 10
- net MRD: track 0.00 -> 159.0 mm, vias 0 -> 8
- net /MA5: track 0.00 -> 158.6 mm, vias 0 -> 12
- net /MA4: track 0.00 -> 157.7 mm, vias 0 -> 10
- net /MA6: track 0.00 -> 154.2 mm, vias 0 -> 13
- net /MA2: track 0.00 -> 153.4 mm, vias 0 -> 8
- net /MA3: track 0.00 -> 141.5 mm, vias 0 -> 7
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Other:
- rule trace_min: 0.2 -> 0.01

Commit message: Look at all the pretty silkscreen
Routing:
- net SC0: track 207.6 -> 203.2 mm, vias 14 -> 13
- net SC1: track 213.0 -> 209.9 mm, vias 11 -> 10
- net TPB: track 175.0 -> 174.3 mm
- net TPA: track 198.5 -> 199.3 mm
Other:
- board text added: "CLK"
- board text added: "DMA IN"
- board text added: "DMA OUT"
- board text added: "EN"
- board text added: "HIGH MEM"
- board text added: "INT"
- board text added: "LOW MEM"
- board text added: "SC0"
- board text added: "SC1"
- board text added: "SLOT #1"
- board text added: "SLOT #2"
- board text added: "TPA"
- board text added: "TPB"
- board text added: "WE"

Commit message: Added provisions for using separate clock circuit
Parts:
- removed JP1: Enable, Pin_Headers:Pin_Header_Straight_1x02_Pitch2.54mm
- added J8: Conn_01x05, Pin_Headers:Pin_Header_Straight_1x05_Pitch2.54mm, F.Cu at (109.9, 66.0)
- moved J7 1.91 mm to (110.5, 55.2)
Connections:
- X1 pad 14: VCC -> GND
- X1 pad 7: GND -> Net-(J8-Pad2)
Routing:
- net Net-(J8-Pad2): track 0.00 -> 6.24 mm
- net Net-(J8-Pad4): track 10.1 -> 6.24 mm
- net CLOCK: track 134.1 -> 131.4 mm
- net VCC: track 400.2 -> 402.2 mm
Other:
- board text added: "BUFFER"
- board text added: "ENABLE"
- board text added: "GND"
- board text added: "INVERTER"
- board text added: "LATCH"
- board text added: "POWER"
- board text added: "RCA CDP1802"
- board text added: "STATUS"
- board text added: "USER INTERFACE"
- board text removed: "EN"
