File: RC1802 CPU/RC1802 CPU.sch (KiCad schematic (older format))
At the start: 54 parts, among them J1 Mount, J2 Mount, J3 Mount, J4 Mount, J5 Expansion, J6 UI_Connector, J7 BARREL_JACK, J8 ClockPort, J9 Q_Connector, U1 74LS04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

Commit message: CPU revision D errata for shorted pins
Other:
- note removed: "RC1802 CPU board"
Changed lines of the file:
@@
 encoding utf-8
 Sheet 1 1
-Title ""
+Title "RC1802 CPU"
 Date ""
-Rev ""
+Rev "F"
 Comp ""
 Comment1 ""
@@
 Text GLabel 13125 4725 2    60   Input ~ 0
 CLOCK_OUT
-Text Notes 12200 10925 0    60   ~ 0
-RC1802 CPU board
 Wire Wire Line
 	4225 1175 4225 1300
